Commit message: Adds first running urdf file of dingo.

File: dingo_fabrics/urdf/dingo_o.urdf (robot description, URDF)
Before this commit: robot dingo, 15 links, 14 joints
Links:
- added link base_link_theta, mass 1.0
- added link base_link_x, mass 1.0
- added link base_link_y, mass 1.0
- added link world, mass 1.0
- link chassis_link: geometry collision mesh filename=meshes/omni_chassis_collision.stl; visual mesh filename=meshes/omni_chassis.dae
Joints:
- added joint base_chassis_joint: type fixed, parent base_link_theta, child base_link, origin xyz=0 0 0 rpy=0 0 0, axis 0 1 0
- added joint joint_theta: type revolute, parent base_link_y, child base_link_theta, origin xyz=0 0 0 rpy=0 0 0, axis 0 0 1, limit lower=-50 upper=50 effort=100 velocity=2
- added joint joint_x: type prismatic, parent world, child base_link_x, origin xyz=0 0 0 rpy=0 0 0, axis 1 0 0, limit lower=-50 upper=50 effort=100 velocity=2
- added joint joint_y: type prismatic, parent base_link_x, child base_link_y, origin xyz=0 0 0 rpy=0 0 0, axis 0 1 0, limit lower=-50 upper=50 effort=100 velocity=2
- joint front_left_wheel: type continuous -> fixed
- joint front_right_wheel: type continuous -> fixed
- joint rear_left_wheel: type continuous -> fixed
- joint rear_right_wheel: type continuous -> fixed
